Commit message: Rebuild hand_v2 bundle from the mirrored description; drop joint calibration, add direct motor control

File: orca_ui/models/hand_v2/left/hand.urdf (robot description, URDF)
Before this commit: robot orcahand_left, 24 links, 23 joints
Links:
- link carpals: mass 0.8542565487567293 -> 0.13538810897856451
- link index_ap: mass 0.004581542163025142 -> 0.004590288233037025
- link thumb_ap: mass 0.007005325272888604 -> 0.007004136465100992
- link thumb_tp: mass 0.007979567574495501 -> 0.00797873207561227
Joints:
- joint index_abd: axis -0.03128510081059521 0.16814409541512249 -0.9852658553123104 -> -8.326672684688674e-17 -3.3306690738754696e-16 -0.9999999999999991; limit lower=-0.436332313 upper=0.5235987756 effort=100 velocity=100 -> lower=-0.4363323129985824 upper=0.5235987755982988 effort=100 velocity=100; origin xyz=0.02724097903991439 -0.0022069668041747375 0.06940680269673632 rpy=-1.6539349343007128 1.3875235793993306 -3.137397887644825 -> xyz=0.027240979039914386 -0.002206966804174762 0.06940680269673646 rpy=1.6538568135338134 -1.3873496487488786 0.0042742186040372054
- joint index_fingertip_fixed: origin xyz=-0.001718 0.0 0.0444 rpy=0 0 0 -> xyz=0.001718 0.0 0.0444 rpy=0 0 0
- joint index_mcp: axis 5.995204332975845e-15 -1.0000000000000038 2.0816681711721685e-17 -> 5.828670879282072e-15 1.0000000000000036 -1.1102230246251565e-16; origin xyz=-0.01915096815087688 2.189902551977232e-18 -0.0009999999999970408 rpy=0.0 -1.5707963267948903 0.0 -> xyz=0.01915096815087666 -4.499288227880137e-18 -0.0009999999999971549 rpy=-2.9439233600320843e-16 1.570796326794891 0.0
- joint index_pip: axis -3.552713678800501e-15 -0.9999999999999964 2.706168622523819e-16 -> -3.608224830031759e-15 0.999999999999996 -2.7755575615628914e-16; origin xyz=0.0014999999999999992 -3.8017921562950314e-18 0.03699999999999992 rpy=3.191891195797317e-16 0.0 6.661338147750924e-15 -> xyz=-0.0015000000000000417 -7.819255613844171e-18 0.037000000000000026 rpy=3.3306690738754617e-16 0.0 -6.77236045021344e-15
- joint middle_abd: axis -6.106226635438361e-16 1.6653345369377348e-16 -0.9999999999999963 -> 1.1102230246251565e-15 2.220446049250313e-16 -0.9999999999999971; origin xyz=0.005706333727246732 -0.004023404072025596 0.07850189342716873 rpy=-1.5707963267947105 1.5681085197468256 -3.141592653589607 -> xyz=0.005706333727246699 -0.004023404072025678 0.07850189342716887 rpy=1.5707963267946425 -1.5681783329169052 2.544631172440859e-13
- joint middle_fingertip_fixed: origin xyz=-0.001718 0.0 0.0444 rpy=0 0 0 -> xyz=0.001718 0.0 0.0444 rpy=0 0 0
- joint middle_mcp: axis 5.773159728050814e-15 -1.000000000000006 -1.476683358925257e-16 -> 6.050715484207103e-15 1.0000000000000058 1.1102230246251565e-16; origin xyz=-0.019866967942905434 2.2433222511080304e-18 -0.000999999999995544 rpy=0.0 -1.5707963267948908 0.0 -> xyz=0.019866967942905277 -1.8423293703642938e-17 -0.0009999999999957202 rpy=0.0 1.5707963267948903 0.0
- joint middle_pip: axis -3.2751579226442118e-15 -0.9999999999999984 7.968885967768458e-17 -> -3.2751579226442118e-15 0.9999999999999977 -4.440892098500626e-16; origin xyz=0.0020000000000000013 -7.514798000251117e-18 0.04000000000000003 rpy=2.3310346708438266e-16 0.0 6.217248937900862e-15 -> xyz=-0.0020000000000000313 -5.598548939047626e-18 0.0400000000000001 rpy=5.551115123125779e-16 -4.440892098500626e-16 -6.550315845288408e-15
- joint pinky_abd: axis -0.13297994090837154 -0.34829476172536833 -0.927904679517606 -> 9.71445146547012e-16 -1.6653345369377348e-16 -0.9999999999999984; origin xyz=-0.03564171604590434 0.0006891586859576484 0.06205424192069404 rpy=1.5294679618327596 1.2029145266720778 -0.22960913173696929 -> xyz=-0.035641716045904354 0.0006891586859576128 0.06205424192069395 rpy=-1.529473573814961 -1.2028622114983025 2.9119895363116646
- joint pinky_fingertip_fixed: origin xyz=-0.002225 -0.0 0.0374 rpy=0 0 0 -> xyz=0.002225 -0.0 0.0374 rpy=0 0 0
- joint pinky_mcp: axis 5.495603971894525e-15 -1.0000000000000044 2.7755575615628914e-17 -> 6.439293542825908e-15 1.0000000000000049 -6.661338147750939e-16; origin xyz=-0.01774999999999982 -5.95919845612908e-17 -0.0009999999999999916 rpy=0.0 -1.5707963267948915 0.0 -> xyz=0.017750000000000075 -4.698582746252626e-17 -0.0010000000000000768 rpy=0.0 1.5707963267948908 0.0
- joint pinky_pip: axis -3.164135620181696e-15 -0.9999999999999976 1.1102230246251565e-16 -> -2.609024107869118e-15 0.9999999999999968 -3.885780586188048e-16; origin xyz=0.0009999999999999979 -1.3225694162272767e-17 0.030999999999999892 rpy=1.3877787807814457e-16 0.0 5.884182030513316e-15 -> xyz=-0.000999999999999998 3.208202345938654e-17 0.030999999999999632 rpy=1.1102230246251565e-16 0.0 -6.217248937900863e-15
- joint ring_abd: axis -0.025208135220825684 -0.17180872948058878 -0.9848077530122064 -> 8.881784197001252e-16 5.551115123125783e-17 -0.9999999999999994; origin xyz=-0.015307722147416563 -0.0032183646651256395 0.07130479703009845 rpy=1.570796326794893 1.4251136941309301 -0.08726646259971993 -> xyz=-0.015307722147416544 -0.003218364665125601 0.07130479703009855 rpy=-1.5707963267948946 -1.4250613342533707 3.054326190990075
- joint ring_fingertip_fixed: origin xyz=-0.001718 0.0 0.0444 rpy=0 0 0 -> xyz=0.001718 0.0 0.0444 rpy=0 0 0
- joint ring_mcp: axis 6.050715484207103e-15 -1.0000000000000036 -5.551115123125783e-17 -> 5.9396931817445875e-15 1.0000000000000042 -1.1102230246251565e-16; origin xyz=-0.01986696794290542 7.724722121653367e-18 -0.0009999999999955448 rpy=0.0 -1.5707963267948908 0.0 -> xyz=0.01986696794290542 3.8657355141463114e-17 -0.00099999999999545 rpy=0.0 1.5707963267948908 0.0
- joint ring_pip: axis -3.4416913763379853e-15 -0.9999999999999967 1.5265566588595902e-16 -> -2.942091015256665e-15 0.999999999999996 -2.220446049250313e-16; origin xyz=0.0020000000000000026 1.0167803431570436e-17 0.04000000000000024 rpy=2.2204460492503052e-16 0.0 6.550315845288409e-15 -> xyz=-0.0019999999999998678 1.5882195667426256e-18 0.040000000000000126 rpy=2.2204460492503052e-16 0.0 -6.217248937900862e-15
- joint thumb_abd: axis 1.27675647831893e-15 0.3420201433256675 -0.9396926207859057 -> -1.4988010832439613e-15 -0.3420201433256641 -0.9396926207859044; origin xyz=-0.008000000000000014 -2.3699749316290387e-17 -0.003850000000000124 rpy=1.2217304763960308 -2.886579864025407e-15 1.9984014443252818e-15 -> xyz=0.007999999999728488 -1.8648424965940806e-17 -0.003850000000000026 rpy=-1.221730476396032 1.9984014443252818e-15 2.3314683517128287e-15
- joint thumb_cmc: axis -2.435551760271437e-15 3.885780586188048e-16 0.9999999999999951 -> -7.771561172376096e-16 -5.412337245047638e-16 0.9999999999999931; origin xyz=0.028398719136200797 0.010997180928709051 0.03058953349163119 rpy=-0.6616685732384568 0.3857244523560657 -1.7091857348501476 -> xyz=0.028398719136200776 0.010997180928709077 0.03058953349163134 rpy=0.6614951404674763 -0.3860568562160207 1.4328677049607634
- joint thumb_dip: axis -8.604228440844963e-16 -0.9999999999999971 -4.440892098500626e-16 -> 4.718447854656915e-16 0.9999999999999946 -3.164135620181696e-15; origin xyz=0.0010000000000000896 -1.3141266374808417e-17 0.03200000000000025 rpy=0.0 0.0 3.885780586188038e-15 -> xyz=-0.0009999999999999985 1.1880660448999647e-16 0.03200000000000021 rpy=0.0 0.0 3.830269434956779e-15
- joint thumb_fingertip_fixed: origin xyz=0.001017 0.0 0.03 rpy=0 0 0 -> xyz=-0.001017 0.0 0.03 rpy=0 0 0
- joint thumb_mcp: axis 3.1086244689504383e-15 -1.0000000000000049 -2.7755575615628914e-16 -> -3.1363800445660672e-15 1.0000000000000027 -2.942091015256665e-15; origin xyz=-0.02800000000000005 7.823464669468643e-17 -3.231584414086884e-18 rpy=-3.1415926535897927 1.570796326794893 0.0 -> xyz=0.027999999999999976 4.673366946417151e-18 1.305542026140606e-16 rpy=-3.1415926535897927 -1.5707963267948921 0.0
- joint tower_fixed: origin xyz=-0.010000000000000018 0.05230000000000584 -2.0816681711721685e-17 rpy=-1.5707963267948966 1.570796326794894 0.0 -> xyz=0.010000000000000018 0.05230000000000584 -2.0816681711721685e-17 rpy=-1.5707963267948966 -1.570796326794894 0.0
- joint wrist: axis -0.9999999999999971 1.767581259681953e-16 -1.318389841742366e-16 -> -0.9999999999999963 1.1270242357758872e-16 -5.94450127715256e-17; origin xyz=4.336808689942018e-19 1.734723475976807e-18 0.04000000000000012 rpy=0.0 2.220446049250313e-16 -1.5707963267948992 -> xyz=-5.551115123125783e-17 2.3418766925686896e-17 0.04000000000000006 rpy=0.0 0.0 1.5707963267948992

File: orca_ui/models/hand_v2/right/hand.urdf (robot description, URDF)
Before this commit: robot orcahand_right, 24 links, 23 joints
Joints:
- joint wrist: origin xyz=5.551115123125783e-17 2.3418766925686896e-17 0.04000000000000006 rpy=-0.610865285723758 0.0 -1.5707963267948992 -> xyz=5.551115123125783e-17 2.3418766925686896e-17 0.04000000000000006 rpy=0.0 0.0 -1.5707963267948992
