Commit message: Read fingertip anchors from the description URDFs instead of deriving them
orcahand_description now owns the {side}_{finger}_fingertip anchor links;
the build reads them from the source URDF and verifies each against the
skin-mesh bbox derivation it previously used to invent them (10 um drift
budget; current drift is sub-micron on every finger). hand.urdf changes
only in element order (fingertip links now flow through the normal
link/joint passes); fingertips.yaml values are identical bar a -0.0
normalization. 152 tests + frontend check-urdf pass.

Co-Authored-By: Claude Fable 5 <noreply@anthropic.com>

File: orca_ui/models/hand_v2/left/hand.urdf (robot description, URDF)
Before this commit: robot orcahand_left, 24 links, 23 joints
Joints:
- joint pinky_fingertip_fixed: origin xyz=0.002225 -0.0 0.0374 rpy=0 0 0 -> xyz=0.002225 0.0 0.0374 rpy=0 0 0

File: orca_ui/models/hand_v2/right/hand.urdf (robot description, URDF)
Before this commit: robot orcahand_right, 24 links, 23 joints
Joints:
- joint pinky_fingertip_fixed: origin xyz=-0.002225 -0.0 0.0374 rpy=0 0 0 -> xyz=-0.002225 0.0 0.0374 rpy=0 0 0
